File: CPC464 Splitter Faceplate A1/CPC464 Splitter Faceplate A1.kicad_pcb (KiCad board)
At the start: 2 copper layers, 82.5 x 40.6 mm, 6 parts, among them M1 Mounting, M2 Mounting, M3 Mounting, M4 Mounting

Commit message: Adjusted cutouts
Parts:
- G***: moved to B.Cu
- G***: moved to F.Cu
- turned G*** to 180 degrees
- turned G*** to 0 degrees
Other:
- outline, holes or cut-outs redrawn
